File: design.kicad_sch (KiCad schematic)
At the start: 0 parts

Commit message: init
Parts:
- added H1: MountingHole, MountingHole:MountingHole_2.7mm_M2.5_ISO7380_Pad, symbol Mechanical:MountingHole
- added J1, J2: BM04B-SRSS-TB_LF__SN_, Snapeda:BM04B-SRSS-TB_LF__SN__JST_BM04B-SRSS-TB_LF__SN_, symbol Snapeda:BM04B-SRSS-TB_LF__SN_
- added SW1, SW2: SW_Push, Snapeda:B3F-4055_SW_B3F-4055, symbol Switch:SW_Push
Connections:
- new net: J1.S1 (SHIELD), J1.S2 (SHIELD)
- new net: J2.S1 (SHIELD), J2.S2 (SHIELD)
- new net B1: J1.2, J2.2, SW1.2, SW2.2
- new net B2: J1.3, J2.3
- new net GND: J1.4, J2.4
- new net VCC: J1.1, J2.1, SW1.1, SW2.1
- no-connect marks 0 -> 2
